File: kicad_power/mdriver_hw_power.kicad_pcb (KiCad board)
At the start: 4 copper layers, 115.4 x 107.7 mm, 65 parts, among them J1 Conn_02x05_Odd_Even, J2 Conn_01x02, M1 Fan, Q1 NMOS, Q2 NMOS, Q3 NMOS, Q4 NMOS, Q5 2N7002E, U7 SFH617A-1X007T

Commit message: finished initial layout of power stage in KiCAD
Parts:
- added C26: 100nF, Capacitor_SMD:C_0402_1005Metric, F.Cu at (139.5, 68.3)
- added C27: 100nF, Capacitor_SMD:C_0402_1005Metric, F.Cu at (139.6, 115.6)
- added C28: 100nF, Capacitor_SMD:C_0402_1005Metric, F.Cu at (139.2, 98.0)
- added C29: 100nF, Capacitor_SMD:C_0402_1005Metric, F.Cu at (154.4, 100.5)
- moved R11 2.37 mm to (138.0, 100.5), turned to 0 degrees
- moved C23 2.09 mm to (153.9, 98.5)
- moved C24 2.09 mm to (153.9, 97.5)
- moved C15 0.91 mm to (138.3, 113.5)
- moved C7 0.90 mm to (137.9, 65.0)
- moved C8 0.90 mm to (137.9, 66.2)
- moved C14 0.90 mm to (138.3, 112.4)
- moved C5 0.79 mm to (73.2, 82.0)
- moved R1 0.79 mm to (71.8, 82.5)
- moved C22 0.73 mm to (154.4, 103.8)
- moved C20 0.69 mm to (156.5, 96.0)
- moved C25 0.50 mm to (140.0, 103.0), turned to 180 degrees
- moved FB1 0.30 mm to (159.9, 96.7)
- moved FB2 0.30 mm to (159.9, 95.2)
- moved R10 0.30 mm to (157.9, 95.2)
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Connections:
- C16 pad 2: Net-(U4-GNDA) -> /isense/in+
- C21 pad 2: Net-(U5-HGND) -> /isense/HGND
- C22 pad 2: Net-(U5-HGND) -> /isense/HGND
- C23 pad 2: Net-(U5-HGND) -> /isense/HGND
- C24 pad 2: Net-(U5-HGND) -> /isense/HGND
- C9 pad 2: Net-(U3-GNDA) -> /legA/OUT
- FB3 pad 2: Net-(U5-HGND) -> /isense/HGND
- R1 pad 1: Net-(R1-Pad1) -> Net-(C5-Pad1)
- U2 pad S1: Net-(R1-Pad1) -> Net-(C5-Pad1)
- U2 pad S2: Net-(C5-Pad1) -> unconnected-(U2-PadS2)
- U3 pad 14: Net-(U3-GNDA) -> /legA/OUT
- U4 pad 14: Net-(U4-GNDA) -> /isense/in+
- U5 pad 2: unconnected-(U5-DCDC_HGND-Pad2) -> /isense/HGND
- U5 pad 3: unconnected-(U5-HLDO_IN-Pad3) -> Net-(U5-DCDC_OUT)
- U5 pad 8: Net-(U5-HGND) -> /isense/HGND
Routing:
- net /legA/OUT: track 0.00 -> 13.9 mm, vias 0 -> 1
- net /isense/in+: track 4.96 -> 18.7 mm, vias 16 -> 17
- net /isense/HGND: track 0.00 -> 9.76 mm
- net Net-(U5-DCDC_OUT): track 0.00 -> 7.80 mm, vias 0 -> 2
- net Net-(U5-HGND): track 6.66 -> 0.00 mm
- net Net-(U5-DCDC_IN): track 2.13 -> 7.47 mm
- net 3V3: track 5.06 -> 8.54 mm, vias 4 -> 11
- net LEGAH: track 191.3 -> 194.4 mm
- net ISOGND: track 5.87 -> 2.89 mm, vias 0 -> 6
- net Net-(U5-HLDO_OUT): track 0.00 -> 2.57 mm
- net Net-(U3-GNDA): track 2.57 -> 0.00 mm
- net Net-(C5-Pad1): track 0.00 -> 2.10 mm
- net Net-(U4-GNDA): track 2.08 -> 0.00 mm
- net LEGAL: track 186.4 -> 188.1 mm
- net /isense/diag: track 1.97 -> 3.66 mm, vias 0 -> 2
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- added copper zone on F.Cu, net /isense/HGND
- added copper zone on F.Cu, net /isense/in-
- added copper zone on F.Cu, net 3V3
- added copper zone on In1.Cu, net 3V3
- added copper zone on B.Cu, net ISOGND
